File: HallSwitches.kicad_sch (KiCad schematic)
At the start: 108 parts

Commit message: footprints
Parts:
- C1, C10, C11, C12, C13, C14, C15, C16, C17, C18, C19, C2, C20, C21, C22, C23, C24, C25, C26, C27, C28, C29, C3, C30, C31, C32, C33, C34, C35, C36, C4, C5, C6, C7, C8, C9: footprint (none) -> Capacitor_SMD:C_0603_1608Metric
- R1, R2, R3, R4: footprint (none) -> Resistor_SMD:R_0603_1608Metric
Changed lines of the file:
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@@
 			)
 		)
-		(property "Footprint" ""
+		(property "Footprint" "Capacitor_SMD:C_0603_1608Metric"
 			(at 110.49 22.86 0)
 			(effects
@@
 			)
 		)
-		(property "Footprint" ""
+		(property "Footprint" "Capacitor_SMD:C_0603_1608Metric"
 			(at 57.15 25.4 0)
 			(effects
@@
 			)
 		)
-		(property "Footprint" ""
+		(property "Footprint" "Capacitor_SMD:C_0603_1608Metric"
 			(at 110.49 26.67 0)
 			(effects
@@
 			)
 		)
-		(property "Footprint" ""
+		(property "Footprint" "Resistor_SMD:R_0603_1608Metric"
 			(at 39.37 124.46 0)
 			(effects
@@
 			)
 		)
-		(property "Footprint" ""
+		(property "Footprint" "Capacitor_SMD:C_0603_1608Metric"
 			(at 134.62 21.59 0)
 			(effects
@@
 			)
 		)
-		(property "Footprint" ""
+		(property "Footprint" "Capacitor_SMD:C_0603_1608Metric"
 			(at 138.43 101.6 0)
 			(effects
@@
 			)
 		)
-		(property "Footprint" ""
+		(property "Footprint" "Capacitor_SMD:C_0603_1608Metric"
 			(at 237.49 99.06 0)
 			(effects
@@
 			)
 		)
-		(property "Footprint" ""
+		(property "Footprint" "Capacitor_SMD:C_0603_1608Metric"
 			(at 114.3 110.49 0)
 			(effects
@@
 			)
 		)
-		(property "Footprint" ""
+		(property "Footprint" "Capacitor_SMD:C_0603_1608Metric"
 			(at 238.76 31.75 0)
 			(effects
@@
 			)
 		)
-		(property "Footprint" ""
+		(property "Footprint" "Capacitor_SMD:C_0603_1608Metric"
 			(at 134.62 29.21 0)
 			(effects
@@
 			)
 		)
-		(property "Footprint" ""
+		(property "Footprint" "Capacitor_SMD:C_0603_1608Metric"
 			(at 261.62 109.22 0)
 			(effects
@@
 			)
 		)
-		(property "Footprint" ""
+		(property "Footprint" "Capacitor_SMD:C_0603_1608Metric"
 			(at 237.49 106.68 0)
 			(effects
@@
 			)
 		)
-		(property "Footprint" ""
+		(property "Footprint" "Capacitor_SMD:C_0603_1608Metric"
 			(at 262.89 34.29 0)
 			(effects
@@
 			)
 		)
-		(property "Footprint" ""
+		(property "Footprint" "Capacitor_SMD:C_0603_1608Metric"
 			(at 114.3 106.68 0)
 			(effects
@@
 			)
 		)
-		(property "Footprint" ""
+		(property "Footprint" "Capacitor_SMD:C_0603_1608Metric"
 			(at 261.62 105.41 0)
 			(effects
@@
 			)
 		)
-		(property "Footprint" ""
+		(property "Footprint" "Resistor_SMD:R_0603_1608Metric"
 			(at 35.56 44.45 0)
 			(effects
@@
 			)
 		)
-		(property "Footprint" ""
+		(property "Footprint" "Capacitor_SMD:C_0603_1608Metric"
 			(at 262.89 26.67 0)
 			(effects
@@
 			)
 		)
-		(property "Footprint" ""
+		(property "Footprint" "Capacitor_SMD:C_0603_1608Metric"
 			(at 114.3 102.87 0)
 			(effects
@@
 			)
 		)
-		(property "Footprint" ""
+		(property "Footprint" "Capacitor_SMD:C_0603_1608Metric"
 			(at 237.49 95.25 0)
 			(effects
@@
 			)
 		)
-		(property "Footprint" ""
+		(property "Footprint" "Capacitor_SMD:C_0603_1608Metric"
 			(at 184.15 101.6 0)
 			(effects
@@
 			)
 		)
-		(property "Footprint" ""
+		(property "Footprint" "Capacitor_SMD:C_0603_1608Metric"
 			(at 138.43 109.22 0)
 			(effects
@@
 			)
 		)
-		(property "Footprint" ""
+		(property "Footprint" "Capacitor_SMD:C_0603_1608Metric"
 			(at 134.62 33.02 0)
 			(effects
@@
 			)
 		)
-		(property "Footprint" ""
+		(property "Footprint" "Capacitor_SMD:C_0603_1608Metric"
 			(at 261.62 101.6 0)
 			(effects
@@
 			)
 		)
-		(property "Footprint" ""
+		(property "Footprint" "Capacitor_SMD:C_0603_1608Metric"
 			(at 110.49 19.05 0)
 			(effects
@@
 			)
 		)
-		(property "Footprint" ""
+		(property "Footprint" "Capacitor_SMD:C_0603_1608Metric"
 			(at 238.76 24.13 0)
 			(effects
@@
 			)
 		)
-		(property "Footprint" ""
+		(property "Footprint" "Capacitor_SMD:C_0603_1608Metric"
 			(at 138.43 113.03 0)
 			(effects
@@
 			)
 		)
-		(property "Footprint" ""
+		(property "Footprint" "Capacitor_SMD:C_0603_1608Metric"
 			(at 60.96 105.41 0)
 			(effects
@@
 			)
 		)
-		(property "Footprint" ""
+		(property "Footprint" "Capacitor_SMD:C_0603_1608Metric"
 			(at 110.49 30.48 0)
 			(effects
@@
 			)
 		)
-		(property "Footprint" ""
+		(property "Footprint" "Resistor_SMD:R_0603_1608Metric"
 			(at 162.56 120.65 0)
 			(effects
@@
 			)
 		)
-		(property "Footprint" ""
+		(property "Footprint" "Capacitor_SMD:C_0603_1608Metric"
 			(at 238.76 27.94 0)
 			(effects
@@
 			)
 		)
-		(property "Footprint" ""
+		(property "Footprint" "Capacitor_SMD:C_0603_1608Metric"
 			(at 134.62 25.4 0)
 			(effects
@@
 			)
 		)
-		(property "Footprint" ""
+		(property "Footprint" "Capacitor_SMD:C_0603_1608Metric"
 			(at 185.42 30.48 0)
 			(effects
@@
 			)
 		)
-		(property "Footprint" ""
+		(property "Footprint" "Capacitor_SMD:C_0603_1608Metric"
 			(at 261.62 97.79 0)
 			(effects
@@
 			)
 		)
-		(property "Footprint" ""
+		(property "Footprint" "Resistor_SMD:R_0603_1608Metric"
 			(at 163.83 49.53 0)
 			(effects
@@
 			)
 		)
-		(property "Footprint" ""
+		(property "Footprint" "Capacitor_SMD:C_0603_1608Metric"
 			(at 262.89 38.1 0)
 			(effects
@@
 			)
 		)
-		(property "Footprint" ""
+		(property "Footprint" "Capacitor_SMD:C_0603_1608Metric"
 			(at 262.89 30.48 0)
 			(effects
@@
 			)
 		)
-		(property "Footprint" ""
+		(property "Footprint" "Capacitor_SMD:C_0603_1608Metric"
 			(at 138.43 105.41 0)
 			(effects
@@
 			)
 		)
-		(property "Footprint" ""
+		(property "Footprint" "Capacitor_SMD:C_0603_1608Metric"
 			(at 238.76 35.56 0)
 			(effects
@@
 			)
 		)
-		(property "Footprint" ""
+		(property "Footprint" "Capacitor_SMD:C_0603_1608Metric"
 			(at 114.3 99.06 0)
 			(effects
@@
 			)
 		)
-		(property "Footprint" ""
+		(property "Footprint" "Capacitor_SMD:C_0603_1608Metric"
 			(at 237.49 102.87 0)
 			(effects

Commit message: sync
Changed lines of the file:
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@@
+	)
+	(label "IO4_INT"
+		(at 21.59 33.02 0)
+		(effects
+			(font
+				(size 1.27 1.27)
+			)
+			(justify left bottom)
+		)
 	)
 	(label "IO4_INT"
@@
 	)
 	(label "SDA"
+		(at 21.59 20.32 0)
+		(effects
+			(font
+				(size 1.27 1.27)
+			)
+			(justify left bottom)
+		)
+	)
+	(label "SDA"
 		(at 160.02 113.03 180)
 		(effects
@@
 			)
 			(justify right bottom)
+		)
+	)
+	(label "IO3_INT"
+		(at 21.59 30.48 0)
+		(effects
+			(font
+				(size 1.27 1.27)
+			)
+			(justify left bottom)
 		)
 	)
@@
 		)
 	)
+	(label "SCL"
+		(at 21.59 22.86 0)
+		(effects
+			(font
+				(size 1.27 1.27)
+			)
+			(justify left bottom)
+		)
+	)
 	(label "3V3"
 		(at 35.56 46.99 270)
@@
 	)
 	(label "IO2_INT"
+		(at 21.59 27.94 0)
+		(effects
+			(font
+				(size 1.27 1.27)
+			)
+			(justify left bottom)
+		)
+	)
+	(label "IO2_INT"
 		(at 161.29 46.99 180)
 		(effects
@@
 			)
 			(justify right bottom)
+		)
+	)
+	(label "3V3"
+		(at 21.59 17.78 0)
+		(effects
+			(font
+				(size 1.27 1.27)
+			)
+			(justify left bottom)
+		)
+	)
+	(label "IO1_INT"
+		(at 21.59 25.4 0)
+		(effects
+			(font
+				(size 1.27 1.27)
+			)
+			(justify left bottom)
 		)
 	)
@@
 		)
 	)
+	(hierarchical_label "SDA"
+		(shape input)
+		(at 21.59 20.32 180)
+		(effects
+			(font
+				(size 1.27 1.27)
+			)
+			(justify right)
+		)
+	)
+	(hierarchical_label "IO4_INT"
+		(shape input)
+		(at 21.59 33.02 180)
+		(effects
+			(font
+				(size 1.27 1.27)
+			)
+			(justify right)
+		)
+	)
+	(hierarchical_label "3V3"
+		(shape input)
+		(at 21.59 17.78 180)
+		(effects
+			(font
+				(size 1.27 1.27)
+			)
+			(justify right)
+		)
+	)
+	(hierarchical_label "SCL"
+		(shape input)
+		(at 21.59 22.86 180)
+		(effects
+			(font
+				(size 1.27 1.27)
+			)
+			(justify right)
+		)
+	)
+	(hierarchical_label "IO1_INT"
+		(shape input)
+		(at 21.59 25.4 180)
+		(effects
+			(font
+				(size 1.27 1.27)
+			)
+			(justify right)
+		)
+	)
+	(hierarchical_label "IO2_INT"
+		(shape input)
+		(at 21.59 27.94 180)
+		(effects
+			(font
+				(size 1.27 1.27)
+			)
+			(justify right)
+		)
+	)
+	(hierarchical_label "IO3_INT"
+		(shape input)
+		(at 21.59 30.48 180)
+		(effects
+			(font
+				(size 1.27 1.27)
+			)
+			(justify right)
+		)
+	)

Commit message: sync
Parts:
- removed R1, R2, R3, R4: 10k, Resistor_SMD:R_0603_1608Metric, symbol Device:R_Small
- renumbered C20 to C201, C10 to C202, C5 to C203, C14 to C204, C2 to C205, C11 to C206, C6 to C207, C15 to C208, C3 to C209, C12 to C210, C7 to C211, C16 to C212, C4 to C213, C13 to C214, C8 to C215, C17 to C216, C19 to C217, C29 to C218, C24 to C219, C33 to C220, C21 to C221, C30 to C222, C25 to C223, C34 to C224, C22 to C225, C31 to C226, C26 to C227, C35 to C228, C23 to C229, C32 to C230, C27 to C231, C36 to C232, C9 to C233, C1 to C234, C18 to C235, C28 to C236, H41 to H34, H34 to H35, H42 to H36, H35 to H37, H43 to H38, H36 to H39, H44 to H40, H37 to H41, H45 to H42, H38 to H43, H46 to H44, H39 to H45, H47 to H46, H40 to H47, H57 to H50, H50 to H51, H58 to H52, H51 to H53, H59 to H54, H52 to H55, H60 to H56, H53 to H57, H61 to H58, H54 to H59, H62 to H60, H55 to H61, H63 to H62, H56 to H63
Connections:
- net at H28.2 (OUTPUT): now also IO2.16 (P13); no longer IO2.11 (P07)
- net at H22.2 (OUTPUT): now also IO2.9 (P05); no longer IO2.15 (P12)
- net at H26.2 (OUTPUT): now also IO2.14 (P11); no longer IO2.7 (P03)
- net at H27.2 (OUTPUT): now also IO2.15 (P12); no longer IO2.9 (P05)
- net at IO2.5 (P01): now also H18.2 (OUTPUT); no longer H25.2 (OUTPUT)
- net at IO2.10 (P06): now also H23.2 (OUTPUT); no longer H20.2 (OUTPUT)
- net at H30.2 (OUTPUT): now also IO2.18 (P15); no longer IO2.16 (P13)
- net at IO2.13 (P10): now also H25.2 (OUTPUT); no longer H21.2 (OUTPUT)
- net at H31.2 (OUTPUT): now also IO2.19 (P16); no longer IO2.18 (P15)
- net at IO2.17 (P14): now also H29.2 (OUTPUT); no longer H23.2 (OUTPUT)
- net at H24.2 (OUTPUT): now also IO2.11 (P07); no longer IO2.19 (P16)
- net at IO2.6 (P02): now also H19.2 (OUTPUT); no longer H18.2 (OUTPUT)
- net at IO2.8 (P04): now also H21.2 (OUTPUT); no longer H19.2 (OUTPUT)
- new net: H20.2 (OUTPUT), IO2.7 (P03)
Other:
- moved on the sheet: C202, C204, C206, C208, C210, C212, C214, C216, C217, C218, C219, C220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

Commit message: lcsc part numbers
Parts:
- C201, C202, C203, C204, C205, C206, C207, C208, C209, C210, C211, C212, C213, C214, C215, C216, C217, C218, C219, C220, C221, C222, C223, C224, C225, C226, C227, C228, C229, C230, C231, C232, C233, C234, C235, C236: value 100n -> 100nF; LCSC (none) -> C30926
- H1, H10, H11, H12, H13, H14, H15, H16, H17, H18, H19, H2, H20, H21, H22, H23, H24, H25, H26, H27, H28, H29, H3, H30, H31, H32, H33, H34, H35, H36, H37, H38, H39, H4, H40, H41, H42, H43, H44, H45, H46, H47, H48, H49, H5, H50, H51, H52, H53, H54, H55, H56, H57, H58, H59, H6, H60, H61, H62, H63, H64, H7, H8, H9: LCSC (none) -> C22466024
- IO1, IO2, IO3, IO4: LCSC (none) -> C22396388

Commit message: production ordered
Parts:
- C201, C202, C203, C204, C205, C206, C207, C208, C209, C210, C211, C212, C213, C214, C215, C216, C217, C218, C219, C220, C221, C222, C223, C224, C225, C226, C227, C228, C229, C230, C231, C232, C233, C234, C235, C236: LCSC C30926 -> C14663
Changed lines of the file:
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@@
 			)
 		)
-		(property "LCSC" "C30926"
+		(property "LCSC" "C14663"
 			(at 110.49 22.86 90)
 			(effects
@@
 			)
 		)
-		(property "LCSC" "C30926"
+		(property "LCSC" "C14663"
 			(at 57.15 25.4 90)
 			(effects
@@
 			)
 		)
-		(property "LCSC" "C30926"
+		(property "LCSC" "C14663"
 			(at 110.49 26.67 90)
 			(effects
@@
 			)
 		)
-		(property "LCSC" "C30926"
+		(property "LCSC" "C14663"
 			(at 134.62 21.59 90)
 			(effects
@@
 			)
 		)
-		(property "LCSC" "C30926"
+		(property "LCSC" "C14663"
 			(at 133.35 95.25 90)
 			(effects
@@
 			)
 		)
-		(property "LCSC" "C30926"
+		(property "LCSC" "C14663"
 			(at 232.41 96.52 90)
 			(effects
@@
 			)
 		)
-		(property "LCSC" "C30926"
+		(property "LCSC" "C14663"
 			(at 109.22 104.14 90)
 			(effects
@@
 			)
 		)
-		(property "LCSC" "C30926"
+		(property "LCSC" "C14663"
 			(at 229.87 26.67 90)
 			(effects
@@
 			)
 		)
-		(property "LCSC" "C30926"
+		(property "LCSC" "C14663"
 			(at 134.62 29.21 90)
 			(effects
@@
 			)
 		)
-		(property "LCSC" "C30926"
+		(property "LCSC" "C14663"
 			(at 256.54 106.68 90)
 			(effects
@@
 			)
 		)
-		(property "LCSC" "C30926"
+		(property "LCSC" "C14663"
 			(at 232.41 104.14 90)
 			(effects
@@
 			)
 		)
-		(property "LCSC" "C30926"
+		(property "LCSC" "C14663"
 			(at 254 29.21 90)
 			(effects
@@
 			)
 		)
-		(property "LCSC" "C30926"
+		(property "LCSC" "C14663"
 			(at 109.22 100.33 90)
 			(effects
@@
 			)
 		)
-		(property "LCSC" "C30926"
+		(property "LCSC" "C14663"
 			(at 256.54 102.87 90)
 			(effects
@@
 			)
 		)
-		(property "LCSC" "C30926"
+		(property "LCSC" "C14663"
 			(at 254 21.59 90)
 			(effects
@@
 			)
 		)
-		(property "LCSC" "C30926"
+		(property "LCSC" "C14663"
 			(at 109.22 96.52 90)
 			(effects
@@
 			)
 		)
-		(property "LCSC" "C30926"
+		(property "LCSC" "C14663"
 			(at 232.41 92.71 90)
 			(effects
@@
 			)
 		)
-		(property "LCSC" "C30926"
+		(property "LCSC" "C14663"
 			(at 179.07 99.06 90)
 			(effects
@@
 			)
 		)
-		(property "LCSC" "C30926"
+		(property "LCSC" "C14663"
 			(at 133.35 102.87 90)
 			(effects
@@
 			)
 		)
-		(property "LCSC" "C30926"
+		(property "LCSC" "C14663"
 			(at 134.62 33.02 90)
 			(effects
@@
 			)
 		)
-		(property "LCSC" "C30926"
+		(property "LCSC" "C14663"
 			(at 256.54 99.06 90)
 			(effects
@@
 			)
 		)
-		(property "LCSC" "C30926"
+		(property "LCSC" "C14663"
 			(at 110.49 19.05 90)
 			(effects
@@
 			)
 		)
-		(property "LCSC" "C30926"
+		(property "LCSC" "C14663"
 			(at 229.87 19.05 90)
 			(effects
@@
 			)
 		)
-		(property "LCSC" "C30926"
+		(property "LCSC" "C14663"
 			(at 133.35 106.68 90)
 			(effects
@@
 			)
 		)
-		(property "LCSC" "C30926"
+		(property "LCSC" "C14663"
 			(at 55.88 99.06 90)
 			(effects
@@
 			)
 		)
-		(property "LCSC" "C30926"
+		(property "LCSC" "C14663"
 			(at 110.49 30.48 90)
 			(effects
@@
 			)
 		)
-		(property "LCSC" "C30926"
+		(property "LCSC" "C14663"
 			(at 229.87 22.86 90)
 			(effects
@@
 			)
 		)
-		(property "LCSC" "C30926"
+		(property "LCSC" "C14663"
 			(at 134.62 25.4 90)
 			(effects
@@
 			)
 		)
-		(property "LCSC" "C30926"
+		(property "LCSC" "C14663"
 			(at 176.53 25.4 90)
 			(effects
@@
 			)
 		)
-		(property "LCSC" "C30926"
+		(property "LCSC" "C14663"
 			(at 256.54 95.25 90)
 			(effects
@@
 			)
 		)
-		(property "LCSC" "C30926"
+		(property "LCSC" "C14663"
 			(at 254 33.02 90)
 			(effects
@@
 			)
 		)
-		(property "LCSC" "C30926"
+		(property "LCSC" "C14663"
 			(at 254 25.4 90)
 			(effects
@@
 			)
 		)
-		(property "LCSC" "C30926"
+		(property "LCSC" "C14663"
 			(at 133.35 99.06 90)
 			(effects
@@
 			)
 		)
-		(property "LCSC" "C30926"
+		(property "LCSC" "C14663"
 			(at 229.87 30.48 90)
 			(effects
@@
 			)
 		)
-		(property "LCSC" "C30926"
+		(property "LCSC" "C14663"
 			(at 109.22 92.71 90)
 			(effects
@@
 			)
 		)
-		(property "LCSC" "C30926"
+		(property "LCSC" "C14663"
 			(at 232.41 100.33 90)
 			(effects
