File: echessboard.kicad_pcb (KiCad board)
At the start: 2 copper layers, 205 x 170 mm, 159 parts, among them J1 Conn_01x04_Pin, J3 USB_C_Receptacle_USB2.0_16P, J4 Conn_01x05_Pin, SW1 SW_Push, SW2 SW_Push, SW3 SW_Push, SW4 SW_Push, SW5 SW_Push, U1 STM32F030C6Tx, U3 USBLC6-2P6, U4 XC6206PxxxMR, U5 MCP2221AxST

Commit message: sync
Parts:
- added D11: BlackWins, LED_SMD:LED_0603_1608Metric, F.Cu at (104.8, 80.8)
- added D8: GameRunning, LED_SMD:LED_0603_1608Metric, F.Cu at (102.2, 66.8)
- added R23: 1k, Resistor_SMD:R_0603_1608Metric, B.Cu at (105.5, 103.5)
- added R24: 1k, Resistor_SMD:R_0603_1608Metric, B.Cu at (102.9, 92.5)
- C1, C10, C11, C12, C13, C14, C15, C16, C17, C18, C19, C2, C20, C21, C22, C23, C24, C25, C26, C27, C28, C29, C3, C30, C31, C32, C33, C34, C35, C36, C37, C38, C39, C4, C40, C41, C42, C43, C44, C45, C46, C47, C5, C6, C7, C8, C9, FB1, H1, H10, H11, H12, H13, H14, H15, H16, H17, H18, H19, H2, H20, H21, H22, H23, H24, H25, H26, H27, H28, H29, H3, H30, H31, H32, H33, H34, H35, H36, H37, H38, H39, H4, H40, H41, H42, H43, H44, H45, H46, H47, H48, H49, H5, H50, H51, H52, H53, H54, H55, H56, H57, H58, H59, H6, H60, H61, H62, H63, H64, H7, H8, H9, IO1, IO2, IO3, IO4, J1, J4, R1, R10, R11, R12, R13, R14, R15, R16, R17, R18, R19, R2, R20, R21, R22, R3, R4, R5, R6, R7, R8, R9, U1, U3, U4, U5: moved to B.Cu
- moved H8 313.4 mm to (264.9, 209.9), turned to 180 degrees
- moved H7 306.5 mm to (264.9, 189.9), turned to 180 degrees
- moved H6 300.2 mm to (264.9, 169.9), turned to 180 degrees
- moved H5 294.6 mm to (264.9, 149.9), turned to 180 degrees
- moved H16 291.6 mm to (244.9, 209.9), turned to 180 degrees
- moved H4 289.7 mm to (264.9, 129.9), turned to 180 degrees
- moved C1 288.3 mm to (302.3, 115.0), turned to 180 degrees
- moved C2 288.3 mm to (302.3, 117.5), turned to 180 degrees
- moved C3 288.3 mm to (302.3, 120.0), turned to 180 degrees
- moved C4 288.3 mm to (302.3, 122.5), turned to 180 degrees
- moved C5 288.3 mm to (302.3, 125.0), turned to 180 degrees
- moved C6 288.3 mm to (302.3, 127.5), turned to 180 degrees
- moved C7 288.3 mm to (302.3, 130.1), turned to 180 degrees
- moved C8 288.3 mm to (302.3, 132.6), turned to 180 degrees
- moved C9 288.3 mm to (302.3, 135.1), turned to 180 degrees
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Connections:
- C37 pad 1: Net-(C37-Pad1) -> Net-(U3-VBUS)
- C38 pad 1: Net-(U3-VBUS) -> Net-(U4-VI)
- C39 pad 1: Net-(U3-VBUS) -> Net-(U4-VI)
- FB1 pad 1: Net-(C37-Pad1) -> Net-(U3-VBUS)
- FB1 pad 2: Net-(U3-VBUS) -> Net-(U4-VI)
- J3 pad A4: Net-(C37-Pad1) -> Net-(U3-VBUS)
- J3 pad A9: Net-(C37-Pad1) -> Net-(U3-VBUS)
- J3 pad B4: Net-(C37-Pad1) -> Net-(U3-VBUS)
- J3 pad B9: Net-(C37-Pad1) -> Net-(U3-VBUS)
- U1 pad 25: Net-(D4-A) -> Net-(D11-A)
- U1 pad 26: Net-(D5-A) -> Net-(D4-A)
- U1 pad 27: unconnected-(U1-PB14-Pad27) -> Net-(D5-A)
- U1 pad 28: unconnected-(U1-PB15-Pad28) -> Net-(D8-A)
- U4 pad 3: Net-(U3-VBUS) -> Net-(U4-VI)
Other:
- board text added: "1"
- board text added: "2"
- board text added: "3"
- board text added: "4"
- board text added: "5"
- board text added: "6"
- board text added: "7"
- board text added: "8"
- board text added: "a"
- board text added: "b"
- board text added: "c"
- board text added: "d"
- board text added: "e"
- board text added: "f"
- board text added: "g"
- board text added: "h"

Commit message: sync
Parts:
- SW4, SW5: moved to B.Cu
- moved U4 20.2 mm to (98.2, 200.6), turned to 90 degrees
- moved C37 20.0 mm to (87.4, 201.7), turned to 90 degrees
- moved U1 18.8 mm to (104.2, 187.9), turned to 90 degrees
- moved C39 17.7 mm to (94.7, 200.9), turned to -90 degrees
- moved FB1 17.3 mm to (89.9, 201.0), turned to 90 degrees
- moved C40 14.8 mm to (99.4, 204.1), turned to 0 degrees
- moved C38 13.5 mm to (92.3, 200.4), turned to -90 degrees
- moved D11 12.4 mm to (92.5, 79.0), turned to 180 degrees
- moved D2 9.58 mm to (97.5, 138.2), turned to 180 degrees
- moved D4 6.79 mm to (102.5, 81.5), turned to 180 degrees
- moved D1 5.81 mm to (97.5, 142.2), turned to 180 degrees
- moved D3 5.48 mm to (92.5, 84.0), turned to 180 degrees
- moved D9 5.31 mm to (87.0, 105.0), turned to 180 degrees
- moved D7 5.05 mm to (94.0, 105.0), turned to 180 degrees
- moved D10 5.00 mm to (101.0, 105.0), turned to 180 degrees
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Connections:
- C1 pad 2: /16_HallSwitches/3V3 -> /3V3
- C10 pad 2: /16_HallSwitches/3V3 -> /3V3
- C11 pad 2: /16_HallSwitches/3V3 -> /3V3
- C12 pad 2: /16_HallSwitches/3V3 -> /3V3
- C13 pad 2: /16_HallSwitches/3V3 -> /3V3
- C14 pad 2: /16_HallSwitches/3V3 -> /3V3
- C15 pad 2: /16_HallSwitches/3V3 -> /3V3
- C16 pad 2: /16_HallSwitches/3V3 -> /3V3
- C17 pad 2: /16_HallSwitches/3V3 -> /3V3
- C18 pad 2: /16_HallSwitches/3V3 -> /3V3
- C19 pad 2: /16_HallSwitches/3V3 -> /3V3
- C2 pad 2: /16_HallSwitches/3V3 -> /3V3
- C20 pad 2: /16_HallSwitches/3V3 -> /3V3
- C21 pad 2: /16_HallSwitches/3V3 -> /3V3
- C22 pad 2: /16_HallSwitches/3V3 -> /3V3
- C23 pad 2: /16_HallSwitches/3V3 -> /3V3
- C24 pad 2: /16_HallSwitches/3V3 -> /3V3
- C25 pad 2: /16_HallSwitches/3V3 -> /3V3
- C26 pad 2: /16_HallSwitches/3V3 -> /3V3
- C27 pad 2: /16_HallSwitches/3V3 -> /3V3
- C28 pad 2: /16_HallSwitches/3V3 -> /3V3
- C29 pad 2: /16_HallSwitches/3V3 -> /3V3
- C3 pad 2: /16_HallSwitches/3V3 -> /3V3
- C30 pad 2: /16_HallSwitches/3V3 -> /3V3
- C31 pad 2: /16_HallSwitches/3V3 -> /3V3
- C32 pad 2: /16_HallSwitches/3V3 -> /3V3
- C33 pad 2: /16_HallSwitches/3V3 -> /3V3
- C34 pad 2: /16_HallSwitches/3V3 -> /3V3
- C35 pad 2: /16_HallSwitches/3V3 -> /3V3
- C36 pad 2: /16_HallSwitches/3V3 -> /3V3
- C4 pad 2: /16_HallSwitches/3V3 -> /3V3
- C5 pad 2: /16_HallSwitches/3V3 -> /3V3
- C6 pad 2: /16_HallSwitches/3V3 -> /3V3
- C7 pad 2: /16_HallSwitches/3V3 -> /3V3
- C8 pad 2: /16_HallSwitches/3V3 -> /3V3
- C9 pad 2: /16_HallSwitches/3V3 -> /3V3
- H1 pad 1: /16_HallSwitches/3V3 -> /3V3
- H10 pad 1: /16_HallSwitches/3V3 -> /3V3
- H11 pad 1: /16_HallSwitches/3V3 -> /3V3
- H12 pad 1: /16_HallSwitches/3V3 -> /3V3
- H13 pad 1: /16_HallSwitches/3V3 -> /3V3
- H14 pad 1: /16_HallSwitches/3V3 -> /3V3
- H15 pad 1: /16_HallSwitches/3V3 -> /3V3
- H16 pad 1: /16_HallSwitches/3V3 -> /3V3
- H17 pad 1: /16_HallSwitches/3V3 -> /3V3
- H18 pad 1: /16_HallSwitches/3V3 -> /3V3
- H19 pad 1: /16_HallSwitches/3V3 -> /3V3
- H2 pad 1: /16_HallSwitches/3V3 -> /3V3
- H20 pad 1: /16_HallSwitches/3V3 -> /3V3
- H21 pad 1: /16_HallSwitches/3V3 -> /3V3
- H22 pad 1: /16_HallSwitches/3V3 -> /3V3
- H23 pad 1: /16_HallSwitches/3V3 -> /3V3
- H24 pad 1: /16_HallSwitches/3V3 -> /3V3
- H25 pad 1: /16_HallSwitches/3V3 -> /3V3
- H26 pad 1: /16_HallSwitches/3V3 -> /3V3
- H27 pad 1: /16_HallSwitches/3V3 -> /3V3
- H28 pad 1: /16_HallSwitches/3V3 -> /3V3
- H29 pad 1: /16_HallSwitches/3V3 -> /3V3
- H3 pad 1: /16_HallSwitches/3V3 -> /3V3
- H30 pad 1: /16_HallSwitches/3V3 -> /3V3
- H31 pad 1: /16_HallSwitches/3V3 -> /3V3
- H32 pad 1: /16_HallSwitches/3V3 -> /3V3
- H33 pad 1: /16_HallSwitches/3V3 -> /3V3
- H34 pad 1: /16_HallSwitches/3V3 -> /3V3
- H35 pad 1: /16_HallSwitches/3V3 -> /3V3
- H36 pad 1: /16_HallSwitches/3V3 -> /3V3
- H37 pad 1: /16_HallSwitches/3V3 -> /3V3
- H38 pad 1: /16_HallSwitches/3V3 -> /3V3
- H39 pad 1: /16_HallSwitches/3V3 -> /3V3
- H4 pad 1: /16_HallSwitches/3V3 -> /3V3
- H40 pad 1: /16_HallSwitches/3V3 -> /3V3
- H41 pad 1: /16_HallSwitches/3V3 -> /3V3
- H42 pad 1: /16_HallSwitches/3V3 -> /3V3
- H43 pad 1: /16_HallSwitches/3V3 -> /3V3
- H44 pad 1: /16_HallSwitches/3V3 -> /3V3
- H45 pad 1: /16_HallSwitches/3V3 -> /3V3
- H46 pad 1: /16_HallSwitches/3V3 -> /3V3
- H47 pad 1: /16_HallSwitches/3V3 -> /3V3
- H48 pad 1: /16_HallSwitches/3V3 -> /3V3
- H49 pad 1: /16_HallSwitches/3V3 -> /3V3
- H5 pad 1: /16_HallSwitches/3V3 -> /3V3
- H50 pad 1: /16_HallSwitches/3V3 -> /3V3
- H51 pad 1: /16_HallSwitches/3V3 -> /3V3
- H52 pad 1: /16_HallSwitches/3V3 -> /3V3
- H53 pad 1: /16_HallSwitches/3V3 -> /3V3
- H54 pad 1: /16_HallSwitches/3V3 -> /3V3
- H55 pad 1: /16_HallSwitches/3V3 -> /3V3
- H56 pad 1: /16_HallSwitches/3V3 -> /3V3
- H57 pad 1: /16_HallSwitches/3V3 -> /3V3
- H58 pad 1: /16_HallSwitches/3V3 -> /3V3
- H59 pad 1: /16_HallSwitches/3V3 -> /3V3
- H6 pad 1: /16_HallSwitches/3V3 -> /3V3
- H60 pad 1: /16_HallSwitches/3V3 -> /3V3
- H61 pad 1: /16_HallSwitches/3V3 -> /3V3
- H62 pad 1: /16_HallSwitches/3V3 -> /3V3
- H63 pad 1: /16_HallSwitches/3V3 -> /3V3
- H64 pad 1: /16_HallSwitches/3V3 -> /3V3
- H7 pad 1: /16_HallSwitches/3V3 -> /3V3
- H8 pad 1: /16_HallSwitches/3V3 -> /3V3
- H9 pad 1: /16_HallSwitches/3V3 -> /3V3
- IO1 pad 22: /16_HallSwitches/SCL -> /SDA
- IO1 pad 23: /16_HallSwitches/SDA -> /SCL
- IO1 pad 24: /16_HallSwitches/3V3 -> /3V3
- IO2 pad 21: /16_HallSwitches/3V3 -> /3V3
- IO2 pad 22: /16_HallSwitches/SCL -> /SDA
- IO2 pad 23: /16_HallSwitches/SDA -> /SCL
- IO2 pad 24: /16_HallSwitches/3V3 -> /3V3
- IO3 pad 2: /16_HallSwitches/3V3 -> /3V3
- IO3 pad 22: /16_HallSwitches/SCL -> /SDA
- IO3 pad 23: /16_HallSwitches/SDA -> /SCL
- IO3 pad 24: /16_HallSwitches/3V3 -> /3V3
- IO4 pad 2: /16_HallSwitches/3V3 -> /3V3
- IO4 pad 21: /16_HallSwitches/3V3 -> /3V3
- IO4 pad 22: /16_HallSwitches/SCL -> /SDA
- IO4 pad 23: /16_HallSwitches/SDA -> /SCL
- IO4 pad 24: /16_HallSwitches/3V3 -> /3V3
- R1 pad 2: /16_HallSwitches/3V3 -> /3V3
- R2 pad 2: /16_HallSwitches/3V3 -> /3V3
- R3 pad 2: /16_HallSwitches/3V3 -> /3V3
- R4 pad 2: /16_HallSwitches/3V3 -> /3V3
- U1 pad 10: /IO1_INT -> /16_HallSwitches/IO1_INT
- U1 pad 11: /IO2_INT -> /16_HallSwitches/IO2_INT
- U1 pad 12: /IO3_INT -> /16_HallSwitches/IO3_INT
- U1 pad 13: /IO4_INT -> /16_HallSwitches/IO4_INT
Routing:
- net Net-(U3-VBUS): track 0.00 -> 17.7 mm, vias 0 -> 2
- net /USB_N: track 0.00 -> 13.9 mm, vias 0 -> 2
- net /USB_P: track 0.00 -> 12.3 mm, vias 0 -> 3
- net /3V3: track 0.00 -> 4.85 mm
- net Net-(U4-VI): track 0.00 -> 4.82 mm
- net GND: track 0.00 -> 2.56 mm, vias 0 -> 1
- added copper zone on B.Cu, net GND
- added copper zone on F.Cu, net GND
Other:
- board text added: "Confirm"
- board text added: "Draw"
- board text added: "Illegal"
- board text added: "Promotion"
- board text added: "Start game"
- board text added: "Winner"

Commit message: sync
Parts:
- removed C1, C10, C11, C12, C13, C14, C15, C16, C17, C18, C19, C2, C20, C21, C22, C23, C24, C25, C26, C27, C28, C29, C3, C30, C31, C32, C33, C34, C35, C36, C4, C5, C6, C7, C8, C9: 100n, Capacitor_SMD:C_0603_1608Metric
- removed R1, R2, R3, R4: 10k, Resistor_SMD:R_0603_1608Metric
- added C201: 100n, Capacitor_SMD:C_0603_1608Metric, B.Cu at (135.0, 69.8)
- added C202: 100n, Capacitor_SMD:C_0603_1608Metric, B.Cu at (177.2, 94.6)
- added C203: 100n, Capacitor_SMD:C_0603_1608Metric, B.Cu at (135.0, 89.6)
- added C204: 100n, Capacitor_SMD:C_0603_1608Metric, B.Cu at (176.1, 151.8)
- added C205: 100n, Capacitor_SMD:C_0603_1608Metric, B.Cu at (135.9, 109.9)
- added C206: 100n, Capacitor_SMD:C_0603_1608Metric, B.Cu at (175.2, 189.4)
- added C207: 100n, Capacitor_SMD:C_0603_1608Metric, B.Cu at (132.7, 129.7)
- added C208: 100n, Capacitor_SMD:C_0603_1608Metric, B.Cu at (175.5, 209.6)
- added C209: 100n, Capacitor_SMD:C_0603_1608Metric, B.Cu at (135.2, 150.9)
- added C210: 100n, Capacitor_SMD:C_0603_1608Metric, B.Cu at (174.3, 70.4)
- added C211: 100n, Capacitor_SMD:C_0603_1608Metric, B.Cu at (135.1, 170.2)
- added C212: 100n, Capacitor_SMD:C_0603_1608Metric, B.Cu at (175.9, 109.3)
- added C213: 100n, Capacitor_SMD:C_0603_1608Metric, B.Cu at (135.1, 190.2)
- added C214: 100n, Capacitor_SMD:C_0603_1608Metric, B.Cu at (172.8, 129.9)
- added C215: 100n, Capacitor_SMD:C_0603_1608Metric, B.Cu at (135.0, 209.7)
- added C216: 100n, Capacitor_SMD:C_0603_1608Metric, B.Cu at (175.2, 172.1)
- added C217: 100n, Capacitor_SMD:C_0603_1608Metric, B.Cu at (215.1, 209.9)
- added C218: 100n, Capacitor_SMD:C_0603_1608Metric, B.Cu at (255.3, 209.0)
- added C219: 100n, Capacitor_SMD:C_0603_1608Metric, B.Cu at (216.3, 109.9)
- added C220: 100n, Capacitor_SMD:C_0603_1608Metric, B.Cu at (252.8, 130.2)
- added C221: 100n, Capacitor_SMD:C_0603_1608Metric, B.Cu at (215.1, 151.7)
- added C222: 100n, Capacitor_SMD:C_0603_1608Metric, B.Cu at (255.1, 88.1)
- added C223: 100n, Capacitor_SMD:C_0603_1608Metric, B.Cu at (212.9, 88.8)
- added C224: 100n, Capacitor_SMD:C_0603_1608Metric, B.Cu at (254.6, 171.9)
- added C225: 100n, Capacitor_SMD:C_0603_1608Metric, B.Cu at (215.1, 70.1)
- added C226: 100n, Capacitor_SMD:C_0603_1608Metric, B.Cu at (255.0, 191.5)
- added C227: 100n, Capacitor_SMD:C_0603_1608Metric, B.Cu at (214.8, 171.1)
- added C228: 100n, Capacitor_SMD:C_0603_1608Metric, B.Cu at (256.4, 111.1)
- added C229: 100n, Capacitor_SMD:C_0603_1608Metric, B.Cu at (212.6, 128.8)
- added C230: 100n, Capacitor_SMD:C_0603_1608Metric, B.Cu at (254.9, 149.9)
- added C231: 100n, Capacitor_SMD:C_0603_1608Metric, B.Cu at (215.1, 190.2)
- added C232: 100n, Capacitor_SMD:C_0603_1608Metric, B.Cu at (255.2, 69.6)
- added C233: 100n, Capacitor_SMD:C_0603_1608Metric, B.Cu at (136.3, 145.3)
- added C234: 100n, Capacitor_SMD:C_0603_1608Metric, B.Cu at (176.2, 145.8)
- added C235: 100n, Capacitor_SMD:C_0603_1608Metric, B.Cu at (216.4, 145.5)
- added C236: 100n, Capacitor_SMD:C_0603_1608Metric, B.Cu at (255.8, 145.3)
- moved H57 198.1 mm to (265.0, 210.0), turned to 0 degrees
- moved H1 198.0 mm to (125.0, 210.0), turned to 0 degrees
- moved H64 198.0 mm to (265.0, 70.0), turned to 0 degrees
- moved H8 197.9 mm to (125.0, 70.0), turned to 0 degrees
- moved H49 172.1 mm to (245.0, 210.0), turned to 0 degrees
- moved H58 172.1 mm to (265.0, 190.0), turned to 0 degrees
- moved H63 172.1 mm to (265.0, 90.0), turned to 0 degrees
- moved H9 172.1 mm to (145.0, 210.0), turned to 0 degrees
- moved H56 172.0 mm to (245.0, 70.0), turned to 0 degrees
- moved H2 172.0 mm to (125.0, 190.0), turned to 0 degrees
- moved H16 172.0 mm to (145.0, 70.0), turned to 0 degrees
- moved H7 172.0 mm to (125.0, 90.0), turned to 0 degrees
- moved IO4 168.2 mm to (255.0, 140.0), turned to 0 degrees
- moved H41 152.4 mm to (225.0, 210.0), turned to 0 degrees
- moved H59 152.4 mm to (265.0, 170.0), turned to 0 degrees
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Connections:
- IO2 pad 10: Net-(H20-OUTPUT) -> Net-(H23-OUTPUT)
- IO2 pad 11: Net-(H28-OUTPUT) -> Net-(H24-OUTPUT)
- IO2 pad 13: Net-(H21-OUTPUT) -> Net-(H25-OUTPUT)
- IO2 pad 14: Net-(H29-OUTPUT) -> Net-(H26-OUTPUT)
- IO2 pad 15: Net-(H22-OUTPUT) -> Net-(H27-OUTPUT)
- IO2 pad 16: Net-(H30-OUTPUT) -> Net-(H28-OUTPUT)
- IO2 pad 17: Net-(H23-OUTPUT) -> Net-(H29-OUTPUT)
- IO2 pad 18: Net-(H31-OUTPUT) -> Net-(H30-OUTPUT)
- IO2 pad 19: Net-(H24-OUTPUT) -> Net-(H31-OUTPUT)
- IO2 pad 5: Net-(H25-OUTPUT) -> Net-(H18-OUTPUT)
- IO2 pad 6: Net-(H18-OUTPUT) -> Net-(H19-OUTPUT)
- IO2 pad 7: Net-(H26-OUTPUT) -> Net-(H20-OUTPUT)
- IO2 pad 8: Net-(H19-OUTPUT) -> Net-(H21-OUTPUT)
- IO2 pad 9: Net-(H27-OUTPUT) -> Net-(H22-OUTPUT)
- IO3 pad 10: Net-(H36-OUTPUT) -> Net-(H39-OUTPUT)
- IO3 pad 11: Net-(H44-OUTPUT) -> Net-(H40-OUTPUT)
- IO3 pad 13: Net-(H37-OUTPUT) -> Net-(H41-OUTPUT)
- IO3 pad 14: Net-(H45-OUTPUT) -> Net-(H42-OUTPUT)
- IO3 pad 15: Net-(H38-OUTPUT) -> Net-(H43-OUTPUT)
- IO3 pad 16: Net-(H46-OUTPUT) -> Net-(H44-OUTPUT)
- IO3 pad 17: Net-(H39-OUTPUT) -> Net-(H45-OUTPUT)
- IO3 pad 18: Net-(H47-OUTPUT) -> Net-(H46-OUTPUT)
- IO3 pad 19: Net-(H40-OUTPUT) -> Net-(H47-OUTPUT)
- IO3 pad 5: Net-(H41-OUTPUT) -> Net-(H34-OUTPUT)
- IO3 pad 6: Net-(H34-OUTPUT) -> Net-(H35-OUTPUT)
- IO3 pad 7: Net-(H42-OUTPUT) -> Net-(H36-OUTPUT)
- IO3 pad 8: Net-(H35-OUTPUT) -> Net-(H37-OUTPUT)
- IO3 pad 9: Net-(H43-OUTPUT) -> Net-(H38-OUTPUT)
- IO4 pad 10: Net-(H52-OUTPUT) -> Net-(H55-OUTPUT)
- IO4 pad 11: Net-(H60-OUTPUT) -> Net-(H56-OUTPUT)
- IO4 pad 13: Net-(H53-OUTPUT) -> Net-(H57-OUTPUT)
- IO4 pad 14: Net-(H61-OUTPUT) -> Net-(H58-OUTPUT)
- IO4 pad 15: Net-(H54-OUTPUT) -> Net-(H59-OUTPUT)
- IO4 pad 16: Net-(H62-OUTPUT) -> Net-(H60-OUTPUT)
- IO4 pad 17: Net-(H55-OUTPUT) -> Net-(H61-OUTPUT)
- IO4 pad 18: Net-(H63-OUTPUT) -> Net-(H62-OUTPUT)
- IO4 pad 19: Net-(H56-OUTPUT) -> Net-(H63-OUTPUT)
- IO4 pad 5: Net-(H57-OUTPUT) -> Net-(H50-OUTPUT)
- IO4 pad 6: Net-(H50-OUTPUT) -> Net-(H51-OUTPUT)
- IO4 pad 7: Net-(H58-OUTPUT) -> Net-(H52-OUTPUT)
- IO4 pad 8: Net-(H51-OUTPUT) -> Net-(H53-OUTPUT)
- IO4 pad 9: Net-(H59-OUTPUT) -> Net-(H54-OUTPUT)
Routing:
- net /SDA: track 0.00 -> 204.4 mm, vias 0 -> 5
- net /16_HallSwitches/IO4_INT: track 0.00 -> 202.9 mm, vias 0 -> 2
- net /SCL: track 0.00 -> 195.7 mm, vias 0 -> 5
- net /16_HallSwitches/IO3_INT: track 0.00 -> 163.1 mm, vias 0 -> 2
- net Net-(U1-PB0): track 0.00 -> 152.2 mm
- net Net-(D8-A): track 0.00 -> 132.9 mm, vias 0 -> 1
- net Net-(D3-A): track 0.00 -> 128.9 mm, vias 0 -> 1
- net Net-(D11-A): track 0.00 -> 122.8 mm, vias 0 -> 1
- net /16_HallSwitches/IO2_INT: track 0.00 -> 118.2 mm, vias 0 -> 2
- net Net-(U1-PB1): track 0.00 -> 117.3 mm, vias 0 -> 2
- net Net-(D7-A): track 0.00 -> 90.5 mm, vias 0 -> 1
- net Net-(D9-A): track 0.00 -> 90.2 mm, vias 0 -> 1
- net Net-(D10-A): track 0.00 -> 90.1 mm, vias 0 -> 1
- net Net-(D6-A): track 0.00 -> 85.8 mm, vias 0 -> 1
- net Net-(H57-OUTPUT): track 0.00 -> 85.7 mm
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- removed copper zone on B.Cu, net GND
- removed copper zone on F.Cu, net GND

Commit message: lcsc part numbers
Parts:
- C201, C202, C203, C204, C205, C206, C207, C208, C209, C210, C211, C212, C213, C214, C215, C216, C217, C218, C219, C220, C221, C222, C223, C224, C225, C226, C227, C228, C229, C230, C231, C232, C233, C234, C235, C236, C41, C42, C43, C44, C45, C46, C47: value 100n -> 100nF
- C37, C38: value 1u -> 1uF
- C39, C40: value 10u -> 10uF
- D1: value WhiteMove -> ~
- D10: value RookPromotion -> ~
- D11: value BlackWins -> ~
- D2: value BlackMove -> ~
- D3: value WhiteWins -> ~
- D4: value Draw -> ~
- D5: value IllegalMove -> ~
- D6: value BishopPromotion -> ~
- D7: value Knight Promotion -> ~
- D8: value GameRunning -> ~
- D9: value QueenPromotion -> ~
- FB1: footprint Inductor_SMD:L_1206_3216Metric -> Inductor_SMD:L_0603_1608Metric
- R10, R11, R9: value 3.3k -> 3K3
- R12, R13, R15, R16, R17, R18, R19, R20, R21, R22, R23, R24: value 1k -> 1K
- R14, R5, R6: value 10k -> 10K
- R7, R8: value 5.1k -> 5K1
- moved R22 125.0 mm to (114.0, 215.5), turned to 0 degrees
- moved R14 120.8 mm to (113.9, 210.6), turned to -90 degrees
- moved R6 113.2 mm to (158.8, 146.6), turned to 90 degrees
- moved R5 111.1 mm to (155.6, 146.5), turned to 90 degrees
- moved C41 108.9 mm to (96.1, 205.3), turned to 90 degrees
- moved R8 100.1 mm to (79.4, 207.7)
- moved C43 99.9 mm to (102.7, 197.6), turned to 90 degrees
- moved R7 99.5 mm to (79.4, 204.6)
- moved C42 96.5 mm to (111.5, 185.9)
- moved C47 91.8 mm to (114.5, 190.3)
- moved R21 69.5 mm to (108.3, 137.6), turned to -90 degrees
- moved R19 68.3 mm to (100.5, 143.7), turned to 90 degrees
- moved R20 63.2 mm to (104.1, 83.4)
- moved R12 62.3 mm to (111.4, 105.1)
- moved R16 54.9 mm to (103.4, 105.8), turned to 90 degrees
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Routing:
- net Net-(D4-A): track 0.00 -> 117.2 mm, vias 0 -> 1
- net GND: track 2.56 -> 114.6 mm, vias 1 -> 141
- net /3V3: track 10.7 -> 25.5 mm
- net Net-(R22-Pad1): track 0.00 -> 8.85 mm
- net Net-(R9-Pad1): track 5.27 -> 11.6 mm
- net Net-(R10-Pad1): track 2.12 -> 8.42 mm
- net Net-(R11-Pad1): track 4.22 -> 10.5 mm
- net /RST: track 64.7 -> 68.4 mm, vias 3 -> 5
- net Net-(J3-CC1): track 0.00 -> 3.59 mm, vias 0 -> 1
- net Net-(J3-CC2): track 0.00 -> 3.45 mm, vias 0 -> 1
- net Net-(U1-BOOT0): track 41.6 -> 45.0 mm
- net /SCL: track 195.7 -> 199.0 mm, vias 5 -> 6
- net Net-(D1-K): track 0.00 -> 2.47 mm, vias 0 -> 1
- net Net-(D11-K): track 0.00 -> 2.37 mm, vias 0 -> 1
- net /USB_N: track 13.9 -> 11.7 mm
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- added copper zone on B.Cu, net /3V3
- added copper zone on F.Cu, net GND

Commit message: finalize
Parts:
- added G***: LOGO, chesspieces:wn, F.Cu at (94.0, 109.5)
- added G***: LOGO, chesspieces:wq, F.Cu at (87.0, 109.5)
- added G***: LOGO, symbols:forbidden, F.Cu at (111.5, 140.2)
- added G***: LOGO, chesspieces:wr, F.Cu at (101.0, 109.5)
- added G***: LOGO, chesspieces:wp, F.Cu at (96.5, 201.2)
- added G***: LOGO, chesspieces:wb, F.Cu at (108.0, 109.5)
Connections:
- net /RXTX renamed /MCU_TX
- net /TXRX renamed /MCU_RX
Other:
- outline, holes or cut-outs redrawn
- board text added: "2025"
- board text added: "3V3"
- board text added: "Benjamin Schmid Ties"
- board text added: "Boot"
- board text added: "CLK"
- board text added: "CS"
- board text added: "Confirm move"
- board text added: "DIO"
- board text added: "GND"
- board text added: "MISO"
- board text added: "MOSI"
- board text added: "RST"
- board text added: "Reset"
- board text added: "SCLK"
- board text added: "SPI"
- board text added: "SWD"
- board text added: "echessboard"
- board text removed: "Confirm"
- board text removed: "Illegal"
