File: echessboard.kicad_sch (KiCad schematic)
At the start: 15 parts, among them J1 USB_C_Receptacle_USB2.0_14P, U1 STM32F030C6Tx, U2 FT232RL, U3 USBLC6-2P6, U4 XC6206PxxxMR

Commit message: sync
Parts:
- removed J1: USB_C_Receptacle_USB2.0_14P, symbol Connector:USB_C_Receptacle_USB2.0_14P
- removed U2: FT232RL, Package_SO:SSOP-28_5.3x10.2mm_P0.65mm, symbol Interface_USB:FT232RL
- added C42, C43, C44, C45, C46, C47, C48, C49, C50: 100n, symbol Device:C_Small
- added J2: Conn_01x04_Pin, Connector_PinHeader_2.54mm:PinHeader_1x04_P2.54mm_Vertical, symbol Connector:Conn_01x04_Pin
- added J3: USB_C_Receptacle_USB2.0_16P, Connector_USB:USB_C_Receptacle_HRO_TYPE-C-31-M-12, symbol Connector:USB_C_Receptacle_USB2.0_16P
- added R10, R11, R12, R13, R14, R15, R16, R9: 3.3k, symbol Device:R_Small
- added SW1, SW2, SW3, SW4, SW5, SW6, SW7, SW8: SW_Push, button:TL3305BF160QG, symbol Switch:SW_Push
- added U5: MCP2221AxST, Package_SO:TSSOP-14_4.4x5mm_P0.65mm, symbol Interface_USB:MCP2221AxST
Connections:
- net 3V3: now also C40.1, C41.2, U1.1 (VDD), U1.24 (VDD), U1.48 (VDD), U1.9 (VDDA), U4.2 (VO), C42.2, C43.2, J2.4 (Pin_4), U5.1 (VDD), U5.11 (VUSB)
- net GND: now also U1.23 (VSS), U1.47 (VSS), U1.8 (VSSA), C42.1, C43.1, C44.2, C45.2, C46.2, C47.2, C48.2, C49.2, C50.2, J2.3 (Pin_3), J3.A1 (GND), J3.A12 (GND), J3.B1 (GND), J3.B12 (GND), J3.S1 (SHIELD), SW1.1, SW2.1, SW3.1, SW4.1, SW5.1, SW6.1, SW7.1, SW8.1, U5.14 (VSS)
- net USB_N: now also J3.A7 (D-), J3.B7 (D-), U5.12 (D-)
- net USB_P: now also J3.A6 (D+), J3.B6 (D+), U5.13 (D+)
- net at C37.1, FB1.1: now also J3.A4 (VBUS), J3.A9 (VBUS), J3.B4 (VBUS), J3.B9 (VBUS)
- net at R7.1: now also J3.A5 (CC1)
- net at R8.1: now also J3.B5 (CC2)
- net at U1.18 (PB0): now also C44.1, R9.2
- net at U1.19 (PB1): now also C45.1, R10.2
- net at U1.20 (PB2): now also C46.1, R11.2
- net RXTX: now reaches U1.30 (PA9)
- net RXTX: now also U5.5 (URx)
- net TXRX: now reaches U1.31 (PA10)
- net TXRX: now also U5.6 (UTx)
- net SWDIO: now reaches U1.34 (PA13)
- net SWDIO: now also J2.2 (Pin_2)
- net SWCLK: now reaches U1.37 (PA14)
- net SWCLK: now also J2.1 (Pin_1)
- net at U1.39 (PB3): now also C47.1, R12.2
- net at U1.40 (PB4): now also C48.1, R13.2
- net at U1.41 (PB5): now also C49.1, R14.2
- net at U1.42 (PB6): now also C50.1, R15.2
- new net: R13.1, SW5.2
- new net: R16.1, SW8.2
- new net: R9.1, SW1.2
- new net: R10.1, SW2.2
- new net: R12.1, SW4.2
- new net: R15.1, SW7.2
- new net: R11.1, SW3.2
- new net: R14.1, SW6.2
- no-connect marks 0 -> 2
Other:
- note added: "Knight"
- note added: "Queen"
- note added: "Start game"
- moved on the sheet: U1

Commit message: footprints
Parts:
- removed C48, C49, C50: 100n, symbol Device:C_Small
- removed J2: Conn_01x04_Pin, Connector_PinHeader_2.54mm:PinHeader_1x04_P2.54mm_Vertical, symbol Connector:Conn_01x04_Pin
- removed SW6, SW7, SW8: SW_Push, button:TL3305BF160QG, symbol Switch:SW_Push
- added D1: WhiteMove, LED_SMD:LED_0603_1608Metric, symbol Device:LED_Small
- added D10: RookPromotion, LED_SMD:LED_0603_1608Metric, symbol Device:LED_Small
- added D2: BlackMove, LED_SMD:LED_0603_1608Metric, symbol Device:LED_Small
- added D3: WhiteWins, LED_SMD:LED_0603_1608Metric, symbol Device:LED_Small
- added D4: Draw, LED_SMD:LED_0603_1608Metric, symbol Device:LED_Small
- added D5: IllegalMove, LED_SMD:LED_0603_1608Metric, symbol Device:LED_Small
- added D6: BishopPromotion, LED_SMD:LED_0603_1608Metric, symbol Device:LED_Small
- added D7: Knight Promotion, LED_SMD:LED_0603_1608Metric, symbol Device:LED_Small
- added D9: QueenPromotion, LED_SMD:LED_0603_1608Metric, symbol Device:LED_Small
- added J1: Conn_01x04_Pin, Connector_PinHeader_2.54mm:PinHeader_1x04_P2.54mm_Vertical, symbol Connector:Conn_01x04_Pin
- added J4: Conn_01x05_Pin, Connector_PinHeader_2.54mm:PinHeader_1x05_P2.54mm_Vertical, symbol Connector:Conn_01x05_Pin
- added R17, R18, R19, R20, R21, R22: 1k, Resistor_SMD:R_0603_1608Metric, symbol Device:R_Small
- C37, C38: footprint (none) -> Capacitor_SMD:C_0805_2012Metric
- C39, C40: footprint (none) -> Capacitor_SMD:C_1206_3216Metric
- C41, C42, C43, C44, C45, C46, C47: footprint (none) -> Capacitor_SMD:C_0603_1608Metric
- FB1: footprint (none) -> Inductor_SMD:L_1206_3216Metric
- R10, R11, R5, R6, R7, R8, R9: footprint (none) -> Resistor_SMD:R_0603_1608Metric
- R12, R13, R15, R16: value 3.3k -> 1k; footprint (none) -> Resistor_SMD:R_0603_1608Metric
- R14: value 3.3k -> 10k; footprint (none) -> Resistor_SMD:R_0603_1608Metric
- SW1, SW2, SW3, SW4, SW5: footprint button:TL3305BF160QG -> Button_Switch_SMD:SW_SPST_TL3342
Connections:
- net 3V3: now also J4.1 (Pin_1), R22.2
- net GND: now also C47.1, R12.1, R13.1, R14.1, R15.1, R16.1, SW4.2, J4.2 (Pin_2), R17.1, R18.1, R19.1, R20.1, R21.1; no longer C47.2, SW4.1, SW5.1
- net SWCLK: now also J4.4 (Pin_4)
- net SWDIO: now also J4.3 (Pin_3)
- net at SW5.2: now also R22.1; no longer R13.1
- net at R13.2: now also D7.1 (K); no longer U1.40 (PB4)
- net at U1.42 (PB6): now also D10.2 (A); no longer R15.2
- net SPI_CS: now reaches U1.14 (PA4)
- net SPI_CS: now also J1.4 (Pin_4)
- net SPI_SCLK: now reaches U1.15 (PA5)
- net SPI_SCLK: now also J1.3 (Pin_3)
- net SPI_MISO: now reaches U1.16 (PA6)
- net SPI_MISO: now also J1.2 (Pin_2)
- net SPI_MOSI: now reaches U1.17 (PA7)
- net SPI_MOSI: now also J1.1 (Pin_1)
- net at U1.21 (PB10): now also D2.2 (A)
- net at U1.22 (PB11): now also D3.2 (A)
- net at U1.25 (PB12): now also D4.2 (A)
- net at U1.26 (PB13): now also D5.2 (A)
- net at U1.41 (PB5): now also D6.2 (A); no longer R14.2
- net at U1.44 (BOOT0): now also R14.2, SW5.1
- net at U1.46 (PB9): now also D1.2 (A)
- net RST: now reaches U1.7 (NRST)
- net RST: now also C47.2, SW4.1, J4.5 (Pin_5)
- net at R16.2: now also D10.1 (K)
- new net: D3.1 (K), R17.2
- new net: D2.1 (K), R18.2
- new net: D1.1 (K), R19.2
- new net: D7.2 (A), U1.40 (PB4)
- new net: D9.2 (A), U1.39 (PB3)
- new net: D6.1 (K), R12.2
- new net: D9.1 (K), R15.2
- new net: D5.1 (K), R21.2
- new net: D4.1 (K), R20.2
Other:
- note added: "Confirm move"
- note added: "CyclePromotion"
- note removed: "Knight"
- note removed: "Queen"
- moved on the sheet: C39, C40, U4

Commit message: sync
Connections:
- net IO1_INT: now also U1.10 (PA0)
- net IO2_INT: now also U1.11 (PA1)
- net IO3_INT: now also U1.12 (PA2)
- net IO4_INT: now also U1.13 (PA3)
- net SCL: now also U1.32 (PA11)
- net SDA: now also U1.33 (PA12)
Other:
- moved on the sheet: J1, R5, R6
Changed lines of the file:
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@@
 	)
 	(junction
-		(at 120.65 101.6)
-		(diameter 0)
-		(color 0 0 0 0)
-	)
-	(junction
 		(at 140.97 85.09)
 		(diameter 0)
@@
 	)
 	(junction
-		(at 231.14 26.67)
+		(at 196.85 115.57)
 		(diameter 0)
 		(color 0 0 0 0)
@@
 	(wire
 		(pts
-			(xy 105.41 101.6) (xy 120.65 101.6)
+			(xy 196.85 124.46) (xy 207.01 124.46)
+		)
+		(stroke
+			(width 0)
+			(type default)
+		)
+	)
+	(wire
+		(pts
+			(xy 196.85 114.3) (xy 196.85 115.57)
 		)
 		(stroke
@@
 	(wire
 		(pts
-			(xy 231.14 35.56) (xy 241.3 35.56)
+			(xy 196.85 121.92) (xy 196.85 124.46)
 		)
 		(stroke
@@
 	(wire
 		(pts
-			(xy 231.14 25.4) (xy 231.14 26.67)
+			(xy 163.83 99.06) (xy 185.42 99.06)
 		)
 		(stroke
@@
 	(wire
 		(pts
-			(xy 231.14 33.02) (xy 231.14 35.56)
+			(xy 163.83 104.14) (xy 185.42 104.14)
 		)
 		(stroke
@@
 	(wire
 		(pts
+			(xy 163.83 101.6) (xy 185.42 101.6)
+		)
+		(stroke
+			(width 0)
+			(type default)
+		)
+	)
+	(wire
+		(pts
 			(xy 105.41 162.56) (xy 105.41 160.02)
 		)
@@
 	(wire
 		(pts
-			(xy 231.14 26.67) (xy 231.14 27.94)
+			(xy 196.85 115.57) (xy 196.85 116.84)
 		)
 		(stroke
@@
 	(wire
 		(pts
-			(xy 236.22 31.75) (xy 241.3 31.75)
+			(xy 201.93 120.65) (xy 207.01 120.65)
 		)
 		(stroke
@@
 	(wire
 		(pts
-			(xy 231.14 26.67) (xy 236.22 26.67)
+			(xy 196.85 115.57) (xy 201.93 115.57)
 		)
 		(stroke
@@
 	(wire
 		(pts
+			(xy 163.83 96.52) (xy 185.42 96.52)
+		)
+		(stroke
+			(width 0)
+			(type default)
+		)
+	)
+	(wire
+		(pts
 			(xy 105.41 160.02) (xy 120.65 160.02)
 		)
@@
 	)
 	(label "IO3_INT"
-		(at 231.14 52.07 0)
+		(at 185.42 101.6 0)
+		(effects
+			(font
+				(size 1.27 1.27)
+			)
+			(justify left bottom)
+		)
+	)
+	(label "SCL"
+		(at 163.83 124.46 0)
 		(effects
 			(font
@@
 	)
 	(label "SPI_SCLK"
-		(at 198.12 109.22 180)
+		(at 228.6 110.49 180)
 		(effects
 			(font
@@
 	)
 	(label "SCL"
-		(at 241.3 35.56 0)
+		(at 207.01 124.46 0)
 		(effects
 			(font
@@
 	)
 	(label "IO1_INT"
-		(at 231.14 46.99 0)
+		(at 185.42 96.52 0)
 		(effects
 			(font
@@
 	)
 	(label "SPI_MOSI"
-		(at 198.12 114.3 180)
+		(at 228.6 115.57 180)
 		(effects
 			(font
@@
 	)
 	(label "SPI_MISO"
-		(at 198.12 111.76 180)
+		(at 228.6 113.03 180)
 		(effects
 			(font
@@
 	)
 	(label "3V3"
-		(at 231.14 25.4 0)
+		(at 196.85 114.3 0)
 		(effects
 			(font
@@
 	)
 	(label "IO4_INT"
-		(at 231.14 54.61 0)
+		(at 185.42 104.14 0)
 		(effects
 			(font
@@
 		)
 	)
+	(label "SDA"
+		(at 163.83 127 0)
+		(effects
+			(font
+				(size 1.27 1.27)
+			)
+			(justify left bottom)
+		)
+	)
 	(label "SWCLK"
 		(at 182.88 147.32 180)
@@
 	)
 	(label "IO2_INT"
-		(at 231.14 49.53 0)
+		(at 185.42 99.06 0)
 		(effects
 			(font
@@
 	)
 	(label "SDA"
-		(at 241.3 31.75 0)
+		(at 207.01 120.65 0)
 		(effects
 			(font
@@
 	)
 	(label "SPI_CS"
-		(at 198.12 106.68 180)
+		(at 228.6 107.95 180)
 		(effects
 			(font
@@
 	(symbol
 		(lib_id "Connector:Conn_01x04_Pin")
-		(at 203.2 111.76 180)
+		(at 233.68 113.03 180)
 		(unit 1)
 		(exclude_from_sim no)
@@
 		(fields_autoplaced yes)
 		(property "Reference" "J1"
-			(at 204.47 109.2199 0)
+			(at 234.95 110.4899 0)
 			(effects
 				(font
@@
 		)
 		(property "Value" "Conn_01x04_Pin"
-			(at 204.47 111.7599 0)
+			(at 234.95 113.0299 0)
 			(effects
 				(font
@@
 		)
 		(property "Footprint" "Connector_PinHeader_2.54mm:PinHeader_1x04_P2.54mm_Vertical"
-			(at 203.2 111.76 0)
+			(at 233.68 113.03 0)
 			(effects
 				(font
@@
 		)
 		(property "Datasheet" "~"
-			(at 203.2 111.76 0)
+			(at 233.68 113.03 0)
 			(effects
 				(font
@@
 		)
 		(property "Description" "Generic connector, single row, 01x04, script generated"
-			(at 203.2 111.76 0)
+			(at 233.68 113.03 0)
 			(effects
 				(font
@@
 	(symbol
 		(lib_id "Device:R_Small")
-		(at 236.22 29.21 0)
+		(at 201.93 118.11 0)
 		(unit 1)
 		(exclude_from_sim no)
@@
 		(dnp no)
 		(property "Reference" "R5"
-			(at 236.982 27.94 0)
+			(at 202.692 116.84 0)
 			(effects
 				(font
@@
 		)
 		(property "Value" "10k"
-			(at 236.982 30.48 0)
+			(at 202.692 119.38 0)
 			(effects
 				(font
@@
 		)
 		(property "Footprint" "Resistor_SMD:R_0603_1608Metric"
-			(at 236.22 29.21 0)
+			(at 201.93 118.11 0)
 			(effects
 				(font
@@
 		)
 		(property "Datasheet" "~"
-			(at 236.22 29.21 0)
+			(at 201.93 118.11 0)
 			(effects
 				(font
@@
 		)
 		(property "Description" "Resistor, small symbol"
-			(at 236.22 29.21 0)
+			(at 201.93 118.11 0)
 			(effects
 				(font
@@
 	(symbol
 		(lib_id "Device:R_Small")
-		(at 231.14 30.48 0)
+		(at 196.85 119.38 0)
 		(unit 1)
 		(exclude_from_sim no)
@@
 		(dnp no)
 		(property "Reference" "R6"
-			(at 231.902 29.21 0)
+			(at 197.612 118.11 0)
 			(effects
 				(font
@@
 		)
 		(property "Value" "10k"
-			(at 231.902 31.75 0)
+			(at 197.612 120.65 0)
 			(effects
 				(font
@@
 		)
 		(property "Footprint" "Resistor_SMD:R_0603_1608Metric"
-			(at 231.14 30.48 0)
+			(at 196.85 119.38 0)
 			(effects
 				(font
@@
 		)
 		(property "Datasheet" "~"
-			(at 231.14 30.48 0)
+			(at 196.85 119.38 0)
 			(effects
 				(font
@@
 		)
 		(property "Description" "Resistor, small symbol"
-			(at 231.14 30.48 0)
+			(at 196.85 119.38 0)
 			(effects
 				(font
@@
 	)
 	(sheet
-		(at 231.14 43.18)
-		(size 12.7 19.05)
+		(at 185.42 92.71)
+		(size 12.7 12.7)
 		(exclude_from_sim no)
 		(in_bom yes)
@@
 		)
 		(property "Sheetname" "16_HallSwitches"
-			(at 231.14 42.4684 0)
+			(at 185.42 91.9984 0)
 			(effects
 				(font
@@
 		)
 		(property "Sheetfile" "HallSwitches.kicad_sch"
-			(at 231.14 62.8146 0)
+			(at 185.42 105.9946 0)
 			(effects
 				(font

Commit message: sync
Parts:
- added D11: BlackWins, LED_SMD:LED_0603_1608Metric, symbol Device:LED_Small
- added D8: GameRunning, LED_SMD:LED_0603_1608Metric, symbol Device:LED_Small
- added R23, R24: 1k, Resistor_SMD:R_0603_1608Metric, symbol Device:R_Small
Connections:
- net GND: now also R23.1, R24.1
- net at C38.1, C39.1, FB1.2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: no longer U3.5 (VBUS)
- net at C37.1, FB1.1, J3.A4 (VBUS)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: now also U3.5 (VBUS)
- net at U1.25 (PB12): now also D11.2 (A); no longer D4.2 (A)
- net at U1.26 (PB13): now also D4.2 (A); no longer D5.2 (A)
- net at U1.27 (PB14): now also D5.2 (A)
- net at U1.28 (PB15): now also D8.2 (A)
- new net: D8.1 (K), R23.2
- new net: D11.1 (K), R24.2
Other:
- moved on the sheet: C37, C38, D1, D10, D2, D3, D4, D5, D6, D7, D9, FB1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

Commit message: sync
Connections:
- net IO1_INT renamed 16_HallSwitches/IO1_INT
- net IO2_INT renamed 16_HallSwitches/IO2_INT
- net IO3_INT renamed 16_HallSwitches/IO3_INT
- net IO4_INT renamed 16_HallSwitches/IO4_INT
Other:
- sheet 16_HallSwitches ports: added 3V3, IO1_INT, IO2_INT, IO3_INT, IO4_INT, SCL, SDA; removed none
- moved on the sheet: J1, J4, R5, R6

Commit message: lcsc part numbers
Parts:
- C37, C38: value 1u -> 1uF; LCSC (none) -> C28323
- C39, C40: value 10u -> 10uF; LCSC (none) -> C89632
- C41, C42, C43, C44, C45, C46, C47: value 100n -> 100nF; LCSC (none) -> C30926
- D1: value WhiteMove -> ~; LCSC (none) -> C2286
- D10: value RookPromotion -> ~; LCSC (none) -> C2286
- D11: value BlackWins -> ~; LCSC (none) -> C2286
- D2: value BlackMove -> ~; LCSC (none) -> C2286
- D3: value WhiteWins -> ~; LCSC (none) -> C2286
- D4: value Draw -> ~; LCSC (none) -> C2286
- D5: value IllegalMove -> ~; LCSC (none) -> C2286
- D6: value BishopPromotion -> ~; LCSC (none) -> C2286
- D7: value Knight Promotion -> ~; LCSC (none) -> C2286
- D8: value GameRunning -> ~; LCSC (none) -> C2286
- D9: value QueenPromotion -> ~; LCSC (none) -> C2286
- FB1: footprint Inductor_SMD:L_1206_3216Metric -> Inductor_SMD:L_0603_1608Metric; LCSC (none) -> C76808
- J3: LCSC (none) -> C165948
- R10, R11, R9: value 3.3k -> 3K3; LCSC (none) -> C22978
- R12, R13, R15, R16, R17, R18, R19, R20, R21, R22, R23, R24: value 1k -> 1K; LCSC (none) -> C21190
- R14, R5, R6: value 10k -> 10K; LCSC (none) -> C2930027
- R7, R8: value 5.1k -> 5K1; LCSC (none) -> C23186

Commit message: finalize
Parts:
- J1, J4: now left out of the parts list
- SW1, SW2, SW3, SW4, SW5: LCSC (none) -> C318884
- U1: LCSC (none) -> C62514
- U3: LCSC (none) -> C15999
- U4: LCSC (none) -> C5446
- U5: LCSC (none) -> C130462
Connections:
- net RXTX renamed MCU_TX
- net TXRX renamed MCU_RX
Changed lines of the file:
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@@
 		)
 	)
+	(label "MCU_TX"
+		(at 163.83 119.38 0)
+		(effects
+			(font
+				(size 1.27 1.27)
+			)
+			(justify left bottom)
+		)
+	)
 	(label "3V3"
 		(at 146.05 80.01 0)
@@
 		)
 	)
-	(label "TXRX"
+	(label "MCU_RX"
 		(at 163.83 121.92 0)
 		(effects
@@
 		)
 	)
-	(label "TXRX"
-		(at 82.55 60.96 0)
-		(effects
-			(font
-				(size 1.27 1.27)
-			)
-			(justify left bottom)
-		)
-	)
 	(label "3V3"
 		(at 72.39 38.1 180)
@@
 		)
 	)
-	(label "RXTX"
-		(at 163.83 119.38 0)
-		(effects
-			(font
-				(size 1.27 1.27)
-			)
-			(justify left bottom)
-		)
-	)
 	(label "RST"
 		(at 195.58 152.4 180)
@@
 		)
 	)
-	(label "RXTX"
-		(at 82.55 58.42 0)
-		(effects
-			(font
-				(size 1.27 1.27)
-			)
-			(justify left bottom)
-		)
-	)
 	(label "USB_N"
 		(at 62.23 63.5 180)
@@
 		)
 	)
+	(label "MCU_TX"
+		(at 82.55 58.42 0)
+		(effects
+			(font
+				(size 1.27 1.27)
+			)
+			(justify left bottom)
+		)
+	)
+	(label "MCU_RX"
+		(at 82.55 60.96 0)
+		(effects
+			(font
+				(size 1.27 1.27)
+			)
+			(justify left bottom)
+		)
+	)
 	(label "USB_P"
 		(at 77.47 27.94 270)
@@
 		(unit 1)
 		(exclude_from_sim no)
-		(in_bom yes)
+		(in_bom no)
 		(on_board yes)
 		(dnp no)
@@
 			)
 		)
-		(property "LCSC" ""
+		(property "LCSC" "C318884 "
 			(at 35.56 135.89 0)
 			(effects
@@
 		(unit 1)
 		(exclude_from_sim no)
-		(in_bom yes)
+		(in_bom no)
 		(on_board yes)
 		(dnp no)
@@
 			)
 		)
-		(property "LCSC" ""
+		(property "LCSC" "C318884 "
 			(at 114.3 93.98 0)
 			(effects
@@
 			)
 		)
-		(property "LCSC" ""
+		(property "LCSC" "C5446"
 			(at 114.3 26.67 0)
 			(effects
@@
 			)
 		)
-		(property "LCSC" ""
+		(property "LCSC" "C318884 "
 			(at 35.56 129.54 0)
 			(effects
@@
 			)
 		)
-		(property "LCSC" ""
+		(property "LCSC" "C62514"
 			(at 148.59 132.08 0)
 			(effects
@@
 			)
 		)
-		(property "LCSC" ""
+		(property "LCSC" "C318884 "
 			(at 35.56 142.24 0)
 			(effects
@@
 			)
 		)
-		(property "LCSC" ""
+		(property "LCSC" "C130462"
 			(at 72.39 63.5 0)
 			(effects
@@
 			)
 		)
-		(property "LCSC" ""
+		(property "LCSC" "C15999"
 			(at 74.93 22.86 0)
 			(effects
@@
 			)
 		)
-		(property "LCSC" ""
+		(property "LCSC" "C318884 "
 			(at 115.57 105.41 0)
 			(effects

Commit message: production ordered
Parts:
- C39, C40: LCSC C89632 -> C13585
- C41, C42, C43, C44, C45, C46, C47: LCSC C30926 -> C14663
- FB1: LCSC C76808 -> C1002
- R14, R5, R6: LCSC C2930027 -> C25804
Changed lines of the file:
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@@
 			)
 		)
-		(property "LCSC" "C89632"
+		(property "LCSC" "C13585"
 			(at 104.14 29.21 0)
 			(effects
@@
 			)
 		)
-		(property "LCSC" "C76808"
+		(property "LCSC" "C1002"
 			(at 92.71 26.67 90)
 			(effects
@@
 			)
 		)
-		(property "LCSC" "C2930027"
+		(property "LCSC" "C25804"
 			(at 219.71 93.98 0)
 			(effects
@@
 			)
 		)
-		(property "LCSC" "C30926"
+		(property "LCSC" "C14663"
 			(at 83.82 123.19 0)
 			(effects
@@
 			)
 		)
-		(property "LCSC" "C30926"
+		(property "LCSC" "C14663"
 			(at 90.17 123.19 0)
 			(effects
@@
 			)
 		)
-		(property "LCSC" "C30926"
+		(property "LCSC" "C14663"
 			(at 69.85 40.64 0)
 			(effects
@@
 			)
 		)
-		(property "LCSC" "C2930027"
+		(property "LCSC" "C25804"
 			(at 224.79 95.25 0)
 			(effects
@@
 			)
 		)
-		(property "LCSC" "C30926"
+		(property "LCSC" "C14663"
 			(at 96.52 123.19 0)
 			(effects
@@
 			)
 		)
-		(property "LCSC" "C89632"
+		(property "LCSC" "C13585"
 			(at 125.73 29.21 0)
 			(effects
@@
 			)
 		)
-		(property "LCSC" "C2930027"
+		(property "LCSC" "C25804"
 			(at 127 106.68 90)
 			(effects
@@
 			)
 		)
-		(property "LCSC" "C30926"
+		(property "LCSC" "C14663"
 			(at 109.22 91.44 0)
 			(effects
@@
 			)
 		)
-		(property "LCSC" "C30926"
+		(property "LCSC" "C14663"
 			(at 143.51 81.28 0)
 			(effects
@@
 			)
 		)
-		(property "LCSC" "C30926"
+		(property "LCSC" "C14663"
 			(at 143.51 85.09 0)
 			(effects
